File: spec/kitest.kicad_sch (KiCad schematic)
At the start: 3 parts, among them J1 Conn_01x02, J2 Conn_01x02, J3 Conn_01x04

Commit message: footprints
Parts:
- J3: footprint (none) -> hello
Changed lines of the file:
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@@
 			)
 		)
-		(property "Footprint" ""
+		(property "Footprint" "hello"
 			(at 107.95 63.5 0)
 			(effects
